File: Weather Station V2.kicad_pcb (KiCad board)
At the start: 4 copper layers, 123.5 x 67.3 mm, 64 parts, among them J1 SOLAR IN, J10 SP13 Socket, J2 18650, J3 Battery_AUX, J4 Conn_01x08_Socket, J5 Conn_01x08_Socket, J6 USB_C, J7 RYLR998, J8 Breakout, J9 SP13 Socket, Q1 AO4842, Q2 DMP2240UDM-7, SW1 LED_ENABLE, SW2 EN/RST, SW3 BOOT, SW4 POWER_SELECT, SW6 POWER, U1 TP4056, U2 DW01A, U3 LDL1117S33R, U4 MT3608, U5 ESP32-S3-WROOM-1U, U7 USBLC6-2SC6

Commit message: - Chnaged to USBLC6-2SC6 for USB ESD protection - Expose 5V rail to Breakout - Fixed missing battery track to power sensors;
- TO DO: open collector mosfet driver to 5V reg
Parts:
- added Q3: BC547, PCM_Package_TO_SOT_THT_AKL:TO-92_Inline_Wide_CBE, F.Cu at (141.0, 133.1)
- added R11: 10K, Resistor_SMD:R_1206_3216Metric, F.Cu at (145.2, 131.9)
- R3: value 1K -> 3K
- moved R3 12.2 mm to (188.9, 110.5)
- moved SW1 4.64 mm to (185.9, 101.4), turned to 0 degrees
Connections:
- net /CHRG renamed /~{CHRG}
- net /STDBY renamed /~{STDBY}
- Q2 pad 3: /~{SENSOR_EN} -> Net-(Q2B-G)
- R10 pad 1: +3V3 -> /Battery_SW
- R10 pad 2: /~{SENSOR_EN} -> Net-(Q2B-G)
Routing:
- net Net-(U1-PROG): track 3.17 -> 16.3 mm, vias 0 -> 2
- net +3V3: track 81.9 -> 73.1 mm
- net Net-(D1-A): track 19.7 -> 15.8 mm
- net /Battery_SW: track 57.8 -> 61.5 mm
- net GND: track 36.1 -> 37.5 mm, vias 18 -> 19
Other:
- board text added: "- +"
