File: Weather Station V2.kicad_sch (KiCad schematic)
At the start: 50 parts, among them J1 SOLAR IN, J2 18650, J3 Battery_AUX, J6 USB_C, J7 RYLR998, J8 Breakout, Q1 AO4842, Q2 DMP2240UDM-7, SW1 LED_ENABLE, SW2 EN/RST, SW3 BOOT, SW4 POWER_SELECT, SW6 POWER, U1 TP4056, U2 DW01A, U3 LDL1117S33R, U5 ESP32-S3-WROOM-1U, U7 USBLC6-2SC6

Commit message: - Localized Libraries
Parts:
- C1, C10, C2, C3, C4, C5, C6, C7: footprint Capacitor_SMD:C_1206_3216Metric -> FootprintsLib:C_1206_3216Metric; symbol Device:C_Small -> SymbolsLib:C_Small
- D1, D2: footprint LED_SMD:LED_1206_3216Metric -> FootprintsLib:LED_1206_3216Metric; symbol Device:LED -> SymbolsLib:LED
- D5: footprint Diode_SMD:D_SMA -> FootprintsLib:D_SMA; symbol Diode:SS34 -> SymbolsLib:SS34
- H1, H2, H3, H4: footprint PCM_SL_Mechanical:MountingHole_3.2mm_Pad -> FootprintsLib:MountingHole_3.2mm_Pad; symbol PCM_SL_Mechanical:MountingHole_M3_3.2mm_Pad -> SymbolsLib:MountingHole_M3_3.2mm_Pad
- J1: footprint TerminalBlock:TerminalBlock_MaiXu_MX126-5.0-02P_1x02_P5.00mm -> FootprintsLib:TerminalBlock_MaiXu_MX126-5.0-02P_1x02_P5.00mm; symbol Connector:Screw_Terminal_01x02 -> SymbolsLib:Screw_Terminal_01x02
- J2: footprint Battery:BatteryHolder_MPD_BH-18650-PC -> FootprintsLib:BatteryHolder_MPD_BH-18650-PC; symbol Connector:Conn_01x02_Socket -> SymbolsLib:Conn_01x02_Socket
- J3: footprint Connector_JST:JST_EH_B2B-EH-A_1x02_P2.50mm_Vertical -> FootprintsLib:JST_EH_B2B-EH-A_1x02_P2.50mm_Vertical; symbol Connector:Conn_01x02_Socket -> SymbolsLib:Conn_01x02_Socket
- J6: footprint Connector_USB:USB_C_Receptacle_GCT_USB4105-xx-A_16P_TopMnt_Horizontal -> FootprintsLib:USB_C_Receptacle_GCT_USB4105-xx-A_16P_TopMnt_Horizontal; symbol Connector:USB_C_Receptacle_USB2.0_16P -> SymbolsLib:USB_C_Receptacle_USB2.0_16P
- J7, J8: footprint Connector_PinSocket_2.54mm:PinSocket_1x05_P2.54mm_Vertical -> FootprintsLib:PinSocket_1x05_P2.54mm_Vertical; symbol Connector:Conn_01x05_Socket -> SymbolsLib:Conn_01x05_Socket
- Q1: footprint Package_SO:SOIC-8_3.9x4.9mm_P1.27mm -> FootprintsLib:SOIC-8_3.9x4.9mm_P1.27mm; symbol Transistor_FET:AO4842 -> SymbolsLib:AO4842
- Q2: footprint Package_TO_SOT_SMD:SOT-23-6_Handsoldering -> FootprintsLib:SOT-23-6_Handsoldering; symbol Transistor_FET:Q_Dual_PMOS_G1S2G2D2S1D1 -> SymbolsLib:Q_Dual_PMOS_G1S2G2D2S1D1
- R1, R14, R15, R16, R2, R3, R4, R5, R6, R7, R8, R9: footprint Resistor_SMD:R_1206_3216Metric -> FootprintsLib:R_1206_3216Metric; symbol Device:R -> SymbolsLib:R
- SW1, SW4, SW6: footprint PCM_SL_Devices:Slide_Switch_SPDT_P3mm_10x5x10mm -> FootprintsLib:Slide_Switch_SPDT_P3mm_10x5x10mm; symbol Switch:SW_SPDT -> SymbolsLib:SW_SPDT
- SW2, SW3: footprint Button_Switch_THT:SW_PUSH_6mm -> FootprintsLib:SW_PUSH_6mm; symbol PCM_SL_Devices:Push_Button -> SymbolsLib:Push_Button
- U1: footprint Package_SO:SOIC-8-1EP_3.9x4.9mm_P1.27mm_EP2.41x3.3mm_ThermalVias -> FootprintsLib:SOIC-8-1EP_3.9x4.9mm_P1.27mm_EP2.41x3.3mm_ThermalVias; symbol Battery_Management:TP4056-42-ESOP8 -> SymbolsLib:TP4056-42-ESOP8
- U2: footprint Package_TO_SOT_SMD:SOT-23-6_Handsoldering -> FootprintsLib:SOT-23-6_Handsoldering; symbol Battery_Management:DW01A -> SymbolsLib:DW01A
- U3: footprint Package_TO_SOT_SMD:SOT-223-3_TabPin2 -> FootprintsLib:SOT-223-3_TabPin2; symbol Regulator_Linear:LM1117MP-3.3 -> SymbolsLib:LM1117MP-3.3
- U5: footprint RF_Module:ESP32-S3-WROOM-1U -> FootprintsLib:ESP32-S3-WROOM-1U; symbol RF_Module:ESP32-S3-WROOM-1 -> SymbolsLib:ESP32-S3-WROOM-1
- U7: footprint Package_TO_SOT_SMD:SOT-23-6 -> FootprintsLib:SOT-23-6; symbol Power_Protection:USBLC6-2SC6 -> SymbolsLib:USBLC6-2SC6

Commit message: - Fixed SCL SDA swap on breakout pins - Added wind speed test point - Regenerated all boards' stiching vias - Fixed wrong pullup on secondary board WSPEED pin (5V --> 3V3)
Parts:
- added TP-WSP1: TP-WSPD, TestPoint:TestPoint_THTPad_D2.0mm_Drill1.0mm, symbol Connector:TestPoint
Connections:
- net W_SPEED: now also TP-WSP1.1
Changed lines of the file:
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@@
 	)
 	(junction
+		(at 97.79 119.38)
+		(diameter 0)
+		(color 0 0 0 0)
+	)
+	(junction
 		(at 39.37 40.64)
 		(diameter 0)
@@
 	(wire
 		(pts
-			(xy 99.06 119.38) (xy 95.25 119.38)
+			(xy 99.06 119.38) (xy 97.79 119.38)
 		)
 		(stroke
@@
 	(wire
 		(pts
+			(xy 97.79 109.22) (xy 97.79 119.38)
+		)
+		(stroke
+			(width 0)
+			(type default)
+		)
+	)
+	(wire
+		(pts
 			(xy 205.74 33.02) (xy 208.28 33.02)
 		)
@@
 	(wire
 		(pts
+			(xy 97.79 119.38) (xy 95.25 119.38)
+		)
+		(stroke
+			(width 0)
+			(type default)
+		)
+	)
+	(wire
+		(pts
 			(xy 99.06 127) (xy 95.25 127)
 		)
@@
 					(unit 1)
 				)
+			)
+		)
+	)
+	(symbol
+		(lib_id "Connector:TestPoint")
+		(at 97.79 109.22 0)
+		(unit 1)
+		(body_style 1)
+		(exclude_from_sim no)
+		(in_bom yes)
+		(on_board yes)
+		(in_pos_files yes)
+		(dnp no)
+		(fields_autoplaced yes)
+		(property "Reference" "TP-WSP1"
+			(at 100.33 104.6479 0)
+			(show_name no)
+			(do_not_autoplace no)
+			(effects
+				(font
+					(size 1.27 1.27)
+				)
+				(justify left)
+			)
+		)
+		(property "Value" "TP-WSPD"
+			(at 100.33 107.1879 0)
+			(show_name no)
+			(do_not_autoplace no)
+			(effects
+				(font
+					(size 1.27 1.27)
+				)
+				(justify left)
+			)
+		)
+		(property "Footprint" "TestPoint:TestPoint_THTPad_D2.0mm_Drill1.0mm"
+			(at 102.87 109.22 0)
+			(hide yes)
+			(show_name no)
+			(do_not_autoplace no)
+			(effects
+				(font
+					(size 1.27 1.27)
+				)
+			)
+		)
+		(property "Datasheet" ""
+			(at 102.87 109.22 0)
+			(hide yes)
+			(show_name no)
+			(do_not_autoplace no)
+			(effects
+				(font
+					(size 1.27 1.27)
+				)
+			)
+		)
+		(property "Description" "test point"
+			(at 97.79 109.22 0)
+			(hide yes)
+			(show_name no)
+			(do_not_autoplace no)
+			(effects
+				(font
+					(size 1.27 1.27)
+				)
+			)
+		)
+		(pin "1"
+		)
+		(instances
+			(project "Weather Station V2"
+				(path "/817e54af-ab8f-4cfe-9b63-ceac8d6d2a44"
+					(reference "TP-WSP1")
+					(unit 1)
+				)

Commit message: Pre-push commit
Parts:
- TP-WSP1: symbol Connector:TestPoint -> Connector_local:TestPoint
Changed lines of the file:
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@@
 	)
 	(symbol
-		(lib_id "power:GND")
+		(lib_id "power_local:GND")
 		(at 203.2 109.22 0)
 		(unit 1)
@@
 	)
 	(symbol
-		(lib_id "power:+5V")
+		(lib_id "power_local:+5V")
 		(at 242.57 133.35 0)
 		(unit 1)
@@
 	)
 	(symbol
-		(lib_id "power:GND")
+		(lib_id "power_local:GND")
 		(at 203.2 80.01 0)
 		(unit 1)
@@
 	)
 	(symbol
-		(lib_id "power:+3V3")
+		(lib_id "power_local:+3V3")
 		(at 78.74 20.32 0)
 		(unit 1)
@@
 	)
 	(symbol
-		(lib_id "power:GND")
+		(lib_id "power_local:GND")
 		(at 247.65 128.27 0)
 		(unit 1)
@@
 	)
 	(symbol
-		(lib_id "power:GND")
+		(lib_id "power_local:GND")
 		(at 41.91 52.07 0)
 		(unit 1)
@@
 	)
 	(symbol
-		(lib_id "power:GND")
+		(lib_id "power_local:GND")
 		(at 176.53 125.73 0)
 		(mirror x)
@@
 	)
 	(symbol
-		(lib_id "power:GND")
+		(lib_id "power_local:GND")
 		(at 186.69 90.17 0)
 		(unit 1)
@@
 	)
 	(symbol
-		(lib_id "power:GND")
+		(lib_id "power_local:GND")
 		(at 99.06 85.09 0)
 		(unit 1)
@@
 	)
 	(symbol
-		(lib_id "power:PWR_FLAG")
+		(lib_id "power_local:PWR_FLAG")
 		(at 245.11 31.75 0)
 		(unit 1)
@@
 	)
 	(symbol
-		(lib_id "power:+3V3")
+		(lib_id "power_local:+3V3")
 		(at 247.65 123.19 0)
 		(unit 1)
@@
 	)
 	(symbol
-		(lib_id "power:GND")
+		(lib_id "power_local:GND")
 		(at 171.45 58.42 0)
 		(unit 1)
@@
 	)
 	(symbol
-		(lib_id "power:GND")
+		(lib_id "power_local:GND")
 		(at 222.25 29.21 0)
 		(unit 1)
@@
 	)
 	(symbol
-		(lib_id "power:PWR_FLAG")
+		(lib_id "power_local:PWR_FLAG")
 		(at 203.2 66.04 0)
 		(unit 1)
@@
 	)
 	(symbol
-		(lib_id "power:+3V3")
+		(lib_id "power_local:+3V3")
 		(at 273.05 35.56 0)
 		(unit 1)
@@
 	)
 	(symbol
-		(lib_id "power:GND")
+		(lib_id "power_local:GND")
 		(at 162.56 119.38 0)
 		(mirror y)
@@
 	)
 	(symbol
-		(lib_id "power:GND")
+		(lib_id "power_local:GND")
 		(at 48.26 187.96 0)
 		(unit 1)
@@
 	)
 	(symbol
-		(lib_id "power:GND")
+		(lib_id "power_local:GND")
 		(at 223.52 66.04 0)
 		(unit 1)
@@
 	)
 	(symbol
-		(lib_id "power:PWR_FLAG")
+		(lib_id "power_local:PWR_FLAG")
 		(at 190.5 48.26 0)
 		(unit 1)
@@
 	)
 	(symbol
-		(lib_id "power:GND")
+		(lib_id "power_local:GND")
 		(at 171.45 143.51 0)
 		(mirror y)
@@
 	)
 	(symbol
-		(lib_id "Connector:TestPoint")
+		(lib_id "Connector_local:TestPoint")
 		(at 97.79 109.22 0)
 		(unit 1)
@@
 	)
 	(symbol
-		(lib_id "power:GND")
+		(lib_id "power_local:GND")
 		(at 229.87 86.36 0)
 		(unit 1)
@@
 	)
 	(symbol
-		(lib_id "power:GND")
+		(lib_id "power_local:GND")
 		(at 208.28 40.64 0)
 		(unit 1)
@@
 	)
 	(symbol
-		(lib_id "power:PWR_FLAG")
+		(lib_id "power_local:PWR_FLAG")
 		(at 245.11 60.96 0)
 		(unit 1)
@@
 	)
 	(symbol
-		(lib_id "power:GND")
+		(lib_id "power_local:GND")
 		(at 213.36 157.48 0)
 		(mirror y)
@@
 	)
 	(symbol
-		(lib_id "power:GND")
+		(lib_id "power_local:GND")
 		(at 255.27 44.45 0)
 		(unit 1)
@@
 	)
 	(symbol
-		(lib_id "power:+3V3")
+		(lib_id "power_local:+3V3")
 		(at 247.65 152.4 0)
 		(unit 1)
@@
 	)
 	(symbol
-		(lib_id "power:+3V3")
+		(lib_id "power_local:+3V3")
 		(at 41.91 33.02 0)
 		(unit 1)
@@
 	)
 	(symbol
-		(lib_id "power:GND")
+		(lib_id "power_local:GND")
 		(at 87.63 25.4 0)
 		(unit 1)
@@
 	)
 	(symbol
-		(lib_id "power:GND")
+		(lib_id "power_local:GND")
 		(at 257.81 142.24 270)
 		(unit 1)
