File: sensors_interface.kicad_sch (KiCad schematic)
At the start: 18 parts, among them J10 SP13 Socket, J4 Conn_01x08_Socket, J5 Conn_01x08_Socket, J9 SP13 Socket, Q2 DMP2240UDM-7, Q3 BC547, U4 MT3608

Commit message: - Changed comment on page 2 - Fixed Q2B PMOS connections (Li mortacci mia!)
Parts:
- added Q4: NMOS, symbol Simulation_SPICE:NMOS
- added Q5: PMOS, symbol Simulation_SPICE:PMOS
Connections:
- net Battery_SW: now also Q2.2 (S); no longer Q2.4 (D)
- net at C9.1, D3.1 (K), L1.1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: now also Q2.4 (D); no longer Q2.2 (S)
Other:
- note added: "Hp: Vbe = 0.7V Vr11 = 3.3 - 0.7 = 2.6V Ib = 2.6 / 10K = 260 uA"
- note removed: "Vbe = 0.7V Vr11 = 3.3 - 0.7 = 2.6V Ib = 2.6 / 10K = 260 uA"
Changed lines of the file:
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@@
 		)
 	)
-	(text "Vbe = 0.7V\nVr11 = 3.3 - 0.7 = 2.6V\nIb = 2.6 / 10K = 260 uA"
+	(text "Hp: Vbe = 0.7V\nVr11 = 3.3 - 0.7 = 2.6V\nIb = 2.6 / 10K = 260 uA"
 		(exclude_from_sim no)
 		(at 47.498 67.818 0)
@@
 		(lib_id "SymbolsLib:Q_Dual_PMOS_G1S2G2D2S1D1")
 		(at 85.09 49.53 0)
+		(mirror x)
 		(unit 2)
 		(body_style 1)
@@
 		(dnp no)
 		(property "Reference" "Q2"
+			(at 90.932 50.8 0)
+			(show_name no)
+			(do_not_autoplace no)
+			(effects
+				(font
+					(size 1.27 1.27)
+				)
+				(justify left)
+			)
+		)
+		(property "Value" "DMP2240UDM-7"
 			(at 90.932 48.26 0)
-			(show_name no)
-			(do_not_autoplace no)
-			(effects
-				(font
-					(size 1.27 1.27)
-				)
-				(justify left)
-			)
-		)
-		(property "Value" "DMP2240UDM-7"
-			(at 90.932 50.8 0)
 			(show_name no)
 			(do_not_autoplace no)
@@
 			)
 		)
-		(property "Datasheet" ""
+		(property "Datasheet" "https://www.mouser.it/datasheet/3/175/1/ds31197.pdf"
 			(at 86.36 49.53 0)
 			(hide yes)
@@
 	)
 	(symbol
+		(lib_id "Simulation_SPICE:PMOS")
+		(at 128.27 38.1 0)
+		(unit 1)
+		(body_style 1)
+		(exclude_from_sim no)
+		(in_bom yes)
+		(on_board yes)
+		(in_pos_files yes)
+		(dnp no)
+		(property "Reference" "Q5"
+			(at 134.62 36.8299 0)
+			(show_name no)
+			(do_not_autoplace no)
+			(effects
+				(font
+					(size 1.27 1.27)
+				)
+				(justify left)
+			)
+		)
+		(property "Value" "PMOS"
+			(at 134.62 39.3699 0)
+			(show_name no)
+			(do_not_autoplace no)
+			(effects
+				(font
+					(size 1.27 1.27)
+				)
+				(justify left)
+			)
+		)
+		(property "Footprint" ""
+			(at 133.35 35.56 0)
+			(hide yes)
+			(show_name no)
+			(do_not_autoplace no)
+			(effects
+				(font
+					(size 1.27 1.27)
+				)
+			)
+		)
+		(property "Datasheet" "https://ngspice.sourceforge.io/docs/ngspice-html-manual/manual.xhtml#cha_MOSFETs"
+			(at 128.27 50.8 0)
+			(hide yes)
+			(show_name no)
+			(do_not_autoplace no)
+			(effects
+				(font
+					(size 1.27 1.27)
+				)
+			)
+		)
+		(property "Description" "P-MOSFET transistor, drain/source/gate"
+			(at 128.27 38.1 0)
+			(hide yes)
+			(show_name no)
+			(do_not_autoplace no)
+			(effects
+				(font
+					(size 1.27 1.27)
+				)
+			)
+		)
+		(property "Sim.Device" "PMOS"
+			(at 128.27 55.245 0)
+			(hide yes)
+			(show_name no)
+			(do_not_autoplace no)
+			(effects
+				(font
+					(size 1.27 1.27)
+				)
+			)
+		)
+		(property "Sim.Type" "VDMOS"
+			(at 128.27 57.15 0)
+			(hide yes)
+			(show_name no)
+			(do_not_autoplace no)
+			(effects
+				(font
+					(size 1.27 1.27)
+				)
+			)
+		)
+		(property "Sim.Pins" "1=D 2=G 3=S"
+			(at 128.27 53.34 0)
+			(hide yes)
+			(show_name no)
+			(do_not_autoplace no)
+			(effects
+				(font
+					(size 1.27 1.27)
+				)
+			)
+		)
+		(pin "1"
+		)
+		(pin "2"
+		)
+		(pin "3"
+		)
+		(instances
+			(project "Weather Station V2"
+				(path "/817e54af-ab8f-4cfe-9b63-ceac8d6d2a44/10b65a9a-b824-4f45-92b4-b4e156b1f43c"
+					(reference "Q5")
+					(unit 1)
+				)
+			)
+		)
+	)
+	(symbol
 		(lib_id "SymbolsLib:BC547")
 		(at 64.77 58.42 0)
@@
 					(unit 1)
 				)
+			)
+		)
+	)
+	(symbol
+		(lib_id "Simulation_SPICE:NMOS")
+		(at 106.68 38.1 0)
+		(unit 1)
+		(body_style 1)
+		(exclude_from_sim no)
+		(in_bom yes)
+		(on_board yes)
+		(in_pos_files yes)
+		(dnp no)
+		(fields_autoplaced yes)
+		(property "Reference" "Q4"
+			(at 113.03 36.8299 0)
+			(show_name no)
+			(do_not_autoplace no)
+			(effects
+				(font
+					(size 1.27 1.27)
+				)
+				(justify left)
+			)
+		)
+		(property "Value" "NMOS"
+			(at 113.03 39.3699 0)
+			(show_name no)
+			(do_not_autoplace no)
+			(effects
+				(font
+					(size 1.27 1.27)
+				)
+				(justify left)
+			)
+		)
+		(property "Footprint" ""
+			(at 111.76 35.56 0)
+			(hide yes)
+			(show_name no)
+			(do_not_autoplace no)
+			(effects
+				(font
+					(size 1.27 1.27)
+				)
+			)
+		)
+		(property "Datasheet" "https://ngspice.sourceforge.io/docs/ngspice-html-manual/manual.xhtml#cha_MOSFETs"
+			(at 106.68 50.8 0)
+			(hide yes)
+			(show_name no)
+			(do_not_autoplace no)
+			(effects
+				(font
+					(size 1.27 1.27)
+				)
+			)
+		)
+		(property "Description" "N-MOSFET transistor, drain/source/gate"
+			(at 106.68 38.1 0)
+			(hide yes)
+			(show_name no)
+			(do_not_autoplace no)
+			(effects
+				(font
+					(size 1.27 1.27)
+				)
+			)
+		)
+		(property "Sim.Device" "NMOS"
+			(at 106.68 55.245 0)
+			(hide yes)
+			(show_name no)
+			(do_not_autoplace no)
+			(effects
+				(font
+					(size 1.27 1.27)
+				)
+			)
+		)
+		(property "Sim.Type" "VDMOS"
+			(at 106.68 57.15 0)
+			(hide yes)
+			(show_name no)
+			(do_not_autoplace no)
+			(effects
+				(font
+					(size 1.27 1.27)
+				)
+			)
+		)
+		(property "Sim.Pins" "1=D 2=G 3=S"
+			(at 106.68 53.34 0)
+			(hide yes)
+			(show_name no)
+			(do_not_autoplace no)
+			(effects
+				(font
+					(size 1.27 1.27)
+				)
+			)
+		)
+		(pin "1"
+		)
+		(pin "2"
+		)
+		(pin "3"
+		)
+		(instances
+			(project "Weather Station V2"
+				(path "/817e54af-ab8f-4cfe-9b63-ceac8d6d2a44/10b65a9a-b824-4f45-92b4-b4e156b1f43c"
+					(reference "Q4")
+					(unit 1)
+				)

Commit message: Pre-push commit
Parts:
- Q4: symbol Simulation_SPICE:NMOS -> Simulation_SPICE_local:NMOS
- Q5: symbol Simulation_SPICE:PMOS -> Simulation_SPICE_local:PMOS
Changed lines of the file:
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@@
 	)
 	(symbol
-		(lib_id "power:+5V")
+		(lib_id "power_local:+5V")
 		(at 234.95 46.99 0)
 		(unit 1)
@@
 	)
 	(symbol
-		(lib_id "power:GND1")
+		(lib_id "power_local:GND1")
 		(at 104.14 147.32 0)
 		(unit 1)
@@
 	)
 	(symbol
-		(lib_id "power:GND1")
+		(lib_id "power_local:GND1")
 		(at 172.72 147.32 0)
 		(unit 1)
@@
 	)
 	(symbol
-		(lib_id "power:GND1")
+		(lib_id "power_local:GND1")
 		(at 63.5 140.97 0)
 		(unit 1)
@@
 	)
 	(symbol
-		(lib_id "Simulation_SPICE:PMOS")
+		(lib_id "Simulation_SPICE_local:PMOS")
 		(at 128.27 38.1 0)
 		(unit 1)
@@
 	)
 	(symbol
-		(lib_id "power:PWR_FLAG")
+		(lib_id "power_local:PWR_FLAG")
 		(at 87.63 57.15 270)
 		(unit 1)
@@
 	)
 	(symbol
-		(lib_id "power:+5V")
+		(lib_id "power_local:+5V")
 		(at 165.1 62.23 0)
 		(unit 1)
@@
 	)
 	(symbol
-		(lib_id "Simulation_SPICE:NMOS")
+		(lib_id "Simulation_SPICE_local:NMOS")
 		(at 106.68 38.1 0)
 		(unit 1)
@@
 	)
 	(symbol
-		(lib_id "power:GND")
+		(lib_id "power_local:GND")
 		(at 67.31 66.04 0)
 		(mirror y)
@@
 	)
 	(symbol
-		(lib_id "power:GND")
+		(lib_id "power_local:GND")
 		(at 234.95 52.07 270)
 		(mirror x)
@@
 	)
 	(symbol
-		(lib_id "power:GND")
+		(lib_id "power_local:GND")
 		(at 121.92 78.74 0)
 		(mirror y)
@@
 	)
 	(symbol
-		(lib_id "power:+3V3")
+		(lib_id "power_local:+3V3")
 		(at 195.58 64.77 0)
 		(mirror y)
