File: _Secondary board/Secondary Board.kicad_pcb (KiCad board)
At the start: 2 copper layers, 47.2 x 47.2 mm, 23 parts, among them IC1 AS5600-ASOT, J1 Conn_01x05_Socket, U1 BME280, U2 VEML7700-TR, U3 HT7533, U4 A3144

Commit message: - Fixed SCL SDA swap on breakout pins - Added wind speed test point - Regenerated all boards' stiching vias - Fixed wrong pullup on secondary board WSPEED pin (5V --> 3V3)
Parts:
- C1, C2, C3, C5, C6: footprint Capacitor_SMD:C_1206_3216Metric_Pad1.33x1.80mm_HandSolder -> FootprintsLib:C_1206_3216Metric_Pad1.33x1.80mm_HandSolder
- H1, H2, H3: footprint MountingHole:MountingHole_3.2mm_M3_ISO7380_Pad -> FootprintsLib:MountingHole_3.2mm_M3_ISO7380_Pad
- IC1: footprint AS5600-ASOT:SOIC127P600X175-8N -> FootprintsLib:SOIC127P600X175-8N
- J1: footprint Connector_Hirose:Hirose_DF13-05P-1.25DSA_1x05_P1.25mm_Vertical -> FootprintsLib:Hirose_DF13-05P-1.25DSA_1x05_P1.25mm_Vertical
- JP2: footprint Jumper:SolderJumper-3_P1.3mm_Open_RoundedPad1.0x1.5mm -> FootprintsLib:SolderJumper-3_P1.3mm_Open_RoundedPad1.0x1.5mm
- R1, R12, R13: footprint Resistor_SMD:R_1206_3216Metric -> FootprintsLib:R_1206_3216Metric
- TP-5V1, TP-GND1, TP-SCL1, TP-SDA1, TP-WSPD1: footprint TestPoint:TestPoint_THTPad_D1.5mm_Drill0.7mm -> FootprintsLib:TestPoint_THTPad_D1.5mm_Drill0.7mm
- U1: footprint Package_LGA:Bosch_LGA-8_2.5x2.5mm_P0.65mm_ClockwisePinNumbering -> FootprintsLib:Bosch_LGA-8_2.5x2.5mm_P0.65mm_ClockwisePinNumbering
- U2: footprint VEML7700-TR:XDCR_VEML7700-TR -> FootprintsLib:XDCR_VEML7700-TR
- U4: footprint Package_TO_SOT_THT:TO-92S -> FootprintsLib:TO-92S
Connections:
- JP2 pad 3: /+5V -> +3V3
Routing:
- net /+5V: track 55.4 -> 28.6 mm
- net +3V3: track 72.5 -> 88.5 mm, vias 6 -> 7
- net GND: vias 133 -> 242
Other:
- board text added: "3V3"
- board text removed: "5V"
