File: _Secondary board/Secondary Board.kicad_sch (KiCad schematic)
At the start: 23 parts, among them IC1 AS5600-ASOT, J1 Conn_01x05_Socket, U1 BME280, U2 VEML7700-TR, U3 HT7533, U4 A3144

Commit message: - Localized Libraries
Parts:
- C1, C2, C3, C5, C6: footprint Capacitor_SMD:C_1206_3216Metric_Pad1.33x1.80mm_HandSolder -> FootprintsLib:C_1206_3216Metric_Pad1.33x1.80mm_HandSolder; symbol PCM_SL_Devices:Capacitor_NP -> SymbolsLib:Capacitor_NP
- H1, H2, H3: footprint MountingHole:MountingHole_3.2mm_M3_ISO7380_Pad -> FootprintsLib:MountingHole_3.2mm_M3_ISO7380_Pad; symbol PCM_SL_Mechanical:MountingHole_M3_3.2mm_Pad -> SymbolsLib:MountingHole_M3_3.2mm_Pad
- IC1: footprint AS5600-ASOT:SOIC127P600X175-8N -> FootprintsLib:SOIC127P600X175-8N; symbol AS5600-ASOT:AS5600-ASOT -> SymbolsLib:AS5600-ASOT
- J1: footprint Connector_Hirose:Hirose_DF13-05P-1.25DSA_1x05_P1.25mm_Vertical -> FootprintsLib:Hirose_DF13-05P-1.25DSA_1x05_P1.25mm_Vertical; symbol Connector:Conn_01x05_Socket -> SymbolsLib:Conn_01x05_Socket
- JP2: footprint Jumper:SolderJumper-3_P1.3mm_Open_RoundedPad1.0x1.5mm -> FootprintsLib:SolderJumper-3_P1.3mm_Open_RoundedPad1.0x1.5mm; symbol Jumper:SolderJumper_3_Open -> SymbolsLib:SolderJumper_3_Open
- R1, R12, R13: footprint Resistor_SMD:R_1206_3216Metric -> FootprintsLib:R_1206_3216Metric; symbol Device:R -> SymbolsLib:R
- TP-5V1, TP-GND1, TP-SCL1, TP-SDA1, TP-WSPD1: footprint TestPoint:TestPoint_THTPad_D1.5mm_Drill0.7mm -> FootprintsLib:TestPoint_THTPad_D1.5mm_Drill0.7mm; symbol Connector:TestPoint -> SymbolsLib:TestPoint
- U1: footprint Package_LGA:Bosch_LGA-8_2.5x2.5mm_P0.65mm_ClockwisePinNumbering -> FootprintsLib:Bosch_LGA-8_2.5x2.5mm_P0.65mm_ClockwisePinNumbering; symbol Sensor:BME280 -> SymbolsLib:BME280
- U2: footprint VEML7700-TR:XDCR_VEML7700-TR -> FootprintsLib:XDCR_VEML7700-TR; symbol VEML7700-TR:VEML7700-TR -> SymbolsLib:VEML7700-TR
- U4: footprint Package_TO_SOT_THT:TO-92S -> FootprintsLib:TO-92S; symbol Sensor_Magnetic:A1302xUA -> SymbolsLib:A1302xUA
Changed lines of the file:
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@@
 	)
 	(symbol
-		(lib_id "Sensor:BME280")
+		(lib_id "SymbolsLib:BME280")
 		(at 46.99 115.57 270)
 		(unit 1)
@@
 			)
 		)
-		(property "Footprint" "Package_LGA:Bosch_LGA-8_2.5x2.5mm_P0.65mm_ClockwisePinNumbering"
+		(property "Footprint" "FootprintsLib:Bosch_LGA-8_2.5x2.5mm_P0.65mm_ClockwisePinNumbering"
 			(at 35.56 153.67 0)
 			(hide yes)
@@
 	)
 	(symbol
-		(lib_id "PCM_SL_Devices:Capacitor_NP")
+		(lib_id "SymbolsLib:Capacitor_NP")
 		(at 68.58 115.57 270)
 		(mirror x)
@@
 			)
 		)
-		(property "Footprint" "Capacitor_SMD:C_1206_3216Metric_Pad1.33x1.80mm_HandSolder"
+		(property "Footprint" "FootprintsLib:C_1206_3216Metric_Pad1.33x1.80mm_HandSolder"
 			(at 64.77 115.57 0)
 			(hide yes)
@@
 	)
 	(symbol
-		(lib_id "Connector:TestPoint")
+		(lib_id "SymbolsLib:TestPoint")
 		(at 217.17 53.34 270)
 		(unit 1)
@@
 			)
 		)
-		(property "Footprint" "TestPoint:TestPoint_THTPad_D1.5mm_Drill0.7mm"
+		(property "Footprint" "FootprintsLib:TestPoint_THTPad_D1.5mm_Drill0.7mm"
 			(at 217.17 58.42 0)
 			(hide yes)
@@
 	)
 	(symbol
-		(lib_id "Connector:TestPoint")
+		(lib_id "SymbolsLib:TestPoint")
 		(at 217.17 60.96 270)
 		(unit 1)
@@
 			)
 		)
-		(property "Footprint" "TestPoint:TestPoint_THTPad_D1.5mm_Drill0.7mm"
+		(property "Footprint" "FootprintsLib:TestPoint_THTPad_D1.5mm_Drill0.7mm"
 			(at 217.17 66.04 0)
 			(hide yes)
@@
 	)
 	(symbol
-		(lib_id "Device:R")
+		(lib_id "SymbolsLib:R")
 		(at 261.62 125.73 180)
 		(unit 1)
@@
 			)
 		)
-		(property "Footprint" "Resistor_SMD:R_1206_3216Metric"
+		(property "Footprint" "FootprintsLib:R_1206_3216Metric"
 			(at 263.398 125.73 90)
 			(hide yes)
@@
 	)
 	(symbol
-		(lib_id "Connector:Conn_01x05_Socket")
+		(lib_id "SymbolsLib:Conn_01x05_Socket")
 		(at 66.04 50.8 180)
 		(unit 1)
@@
 			)
 		)
-		(property "Footprint" "Connector_Hirose:Hirose_DF13-05P-1.25DSA_1x05_P1.25mm_Vertical"
+		(property "Footprint" "FootprintsLib:Hirose_DF13-05P-1.25DSA_1x05_P1.25mm_Vertical"
 			(at 66.04 50.8 0)
 			(hide yes)
@@
 	)
 	(symbol
-		(lib_id "PCM_SL_Mechanical:MountingHole_M3_3.2mm_Pad")
+		(lib_id "SymbolsLib:MountingHole_M3_3.2mm_Pad")
 		(at 92.71 173.99 0)
 		(unit 1)
@@
 			)
 		)
-		(property "Footprint" "MountingHole:MountingHole_3.2mm_M3_ISO7380_Pad"
+		(property "Footprint" "FootprintsLib:MountingHole_3.2mm_M3_ISO7380_Pad"
 			(at 92.71 177.8 0)
 			(hide yes)
@@
 	)
 	(symbol
-		(lib_id "AS5600-ASOT:AS5600-ASOT")
+		(lib_id "SymbolsLib:AS5600-ASOT")
 		(at 171.45 116.84 0)
 		(unit 1)
@@
 			)
 		)
-		(property "Footprint" "AS5600-ASOT:SOIC127P600X175-8N"
+		(property "Footprint" "FootprintsLib:SOIC127P600X175-8N"
 			(at 171.45 116.84 0)
 			(hide yes)
@@
 	)
 	(symbol
-		(lib_id "PCM_SL_Mechanical:MountingHole_M3_3.2mm_Pad")
+		(lib_id "SymbolsLib:MountingHole_M3_3.2mm_Pad")
 		(at 81.28 173.99 0)
 		(unit 1)
@@
 			)
 		)
-		(property "Footprint" "MountingHole:MountingHole_3.2mm_M3_ISO7380_Pad"
+		(property "Footprint" "FootprintsLib:MountingHole_3.2mm_M3_ISO7380_Pad"
 			(at 81.28 177.8 0)
 			(hide yes)
@@
 	)
 	(symbol
-		(lib_id "PCM_SL_Devices:Capacitor_NP")
+		(lib_id "SymbolsLib:Capacitor_NP")
 		(at 104.14 48.26 90)
 		(unit 1)
@@
 			)
 		)
-		(property "Footprint" "Capacitor_SMD:C_1206_3216Metric_Pad1.33x1.80mm_HandSolder"
+		(property "Footprint" "FootprintsLib:C_1206_3216Metric_Pad1.33x1.80mm_HandSolder"
 			(at 107.95 48.26 0)
 			(hide yes)
@@
 	)
 	(symbol
-		(lib_id "PCM_SL_Devices:Capacitor_NP")
+		(lib_id "SymbolsLib:Capacitor_NP")
 		(at 165.1 120.65 90)
 		(unit 1)
@@
 			)
 		)
-		(property "Footprint" "Capacitor_SMD:C_1206_3216Metric_Pad1.33x1.80mm_HandSolder"
+		(property "Footprint" "FootprintsLib:C_1206_3216Metric_Pad1.33x1.80mm_HandSolder"
 			(at 168.91 120.65 0)
 			(hide yes)
@@
 	)
 	(symbol
-		(lib_id "Jumper:SolderJumper_3_Open")
+		(lib_id "SymbolsLib:SolderJumper_3_Open")
 		(at 261.62 134.62 180)
 		(unit 1)
@@
 			)
 		)
-		(property "Footprint" "Jumper:SolderJumper-3_P1.3mm_Open_RoundedPad1.0x1.5mm"
+		(property "Footprint" "FootprintsLib:SolderJumper-3_P1.3mm_Open_RoundedPad1.0x1.5mm"
 			(at 261.62 134.62 0)
 			(hide yes)
@@
 	)
 	(symbol
-		(lib_id "PCM_SL_Devices:Capacitor_NP")
+		(lib_id "SymbolsLib:Capacitor_NP")
 		(at 125.73 114.3 270)
 		(mirror x)
@@
 			)
 		)
-		(property "Footprint" "Capacitor_SMD:C_1206_3216Metric_Pad1.33x1.80mm_HandSolder"
+		(property "Footprint" "FootprintsLib:C_1206_3216Metric_Pad1.33x1.80mm_HandSolder"
 			(at 121.92 114.3 0)
 			(hide yes)
@@
 	)
 	(symbol
-		(lib_id "Connector:TestPoint")
+		(lib_id "SymbolsLib:TestPoint")
 		(at 217.17 58.42 270)
 		(unit 1)
@@
 			)
 		)
-		(property "Footprint" "TestPoint:TestPoint_THTPad_D1.5mm_Drill0.7mm"
+		(property "Footprint" "FootprintsLib:TestPoint_THTPad_D1.5mm_Drill0.7mm"
 			(at 217.17 63.5 0)
 			(hide yes)
@@
 	)
 	(symbol
-		(lib_id "Sensor_Magnetic:A1302xUA")
+		(lib_id "SymbolsLib:A1302xUA")
 		(at 261.62 113.03 90)
 		(mirror x)
@@
 			)
 		)
-		(property "Footprint" "Package_TO_SOT_THT:TO-92S"
+		(property "Footprint" "FootprintsLib:TO-92S"
 			(at 278.638 113.03 0)
 			(hide yes)
@@
 	)
 	(symbol
-		(lib_id "PCM_SL_Devices:Capacitor_NP")
+		(lib_id "SymbolsLib:Capacitor_NP")
 		(at 132.08 48.26 270)
 		(mirror x)
@@
 			)
 		)
-		(property "Footprint" "Capacitor_SMD:C_1206_3216Metric_Pad1.33x1.80mm_HandSolder"
+		(property "Footprint" "FootprintsLib:C_1206_3216Metric_Pad1.33x1.80mm_HandSolder"
 			(at 128.27 48.26 0)
 			(hide yes)
@@
 	)
 	(symbol
-		(lib_id "PCM_SL_Mechanical:MountingHole_M3_3.2mm_Pad")
+		(lib_id "SymbolsLib:MountingHole_M3_3.2mm_Pad")
 		(at 69.85 173.99 0)
 		(unit 1)
@@
 			)
 		)
-		(property "Footprint" "MountingHole:MountingHole_3.2mm_M3_ISO7380_Pad"
+		(property "Footprint" "FootprintsLib:MountingHole_3.2mm_M3_ISO7380_Pad"
 			(at 69.85 177.8 0)
 			(hide yes)
@@
 	)
 	(symbol
-		(lib_id "Device:R")
+		(lib_id "SymbolsLib:R")
 		(at 82.55 60.96 0)
 		(mirror y)
@@
 			)
 		)
-		(property "Footprint" "Resistor_SMD:R_1206_3216Metric"
+		(property "Footprint" "FootprintsLib:R_1206_3216Metric"
 			(at 84.328 60.96 90)
 			(hide yes)
@@
 	)
 	(symbol
-		(lib_id "Connector:TestPoint")
+		(lib_id "SymbolsLib:TestPoint")
 		(at 217.17 55.88 270)
 		(unit 1)
@@
 			)
 		)
-		(property "Footprint" "TestPoint:TestPoint_THTPad_D1.5mm_Drill0.7mm"
+		(property "Footprint" "FootprintsLib:TestPoint_THTPad_D1.5mm_Drill0.7mm"
 			(at 217.17 60.96 0)
 			(hide yes)
@@
 	)
 	(symbol
-		(lib_id "Connector:TestPoint")
+		(lib_id "SymbolsLib:TestPoint")
 		(at 217.17 63.5 270)
 		(unit 1)
@@
 			)
 		)
-		(property "Footprint" "TestPoint:TestPoint_THTPad_D1.5mm_Drill0.7mm"
+		(property "Footprint" "FootprintsLib:TestPoint_THTPad_D1.5mm_Drill0.7mm"
 			(at 217.17 68.58 0)
 			(hide yes)
@@
 	)
 	(symbol
-		(lib_id "Device:R")
+		(lib_id "SymbolsLib:R")
 		(at 73.66 60.96 0)
 		(mirror y)
@@
 			)
 		)
-		(property "Footprint" "Resistor_SMD:R_1206_3216Metric"
+		(property "Footprint" "FootprintsLib:R_1206_3216Metric"
 			(at 75.438 60.96 90)
 			(hide yes)
@@
 	)
 	(symbol
-		(lib_id "VEML7700-TR:VEML7700-TR")
+		(lib_id "SymbolsLib:VEML7700-TR")
 		(at 110.49 119.38 0)
 		(unit 1)
@@
 			)
 		)
-		(property "Footprint" "VEML7700-TR:XDCR_VEML7700-TR"
+		(property "Footprint" "FootprintsLib:XDCR_VEML7700-TR"
 			(at 110.49 119.38 0)
 			(hide yes)

Commit message: - Fixed SCL SDA swap on breakout pins - Added wind speed test point - Regenerated all boards' stiching vias - Fixed wrong pullup on secondary board WSPEED pin (5V --> 3V3)
Connections:
- net +3V3: now also JP2.3 (B)
- net +5V: no longer JP2.3 (B)
Changed lines of the file:
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@@
-	)
-	(junction
-		(at 241.3 110.49)
-		(diameter 0)
-		(color 0 0 0 0)
 	)
 	(junction
@@
 	(wire
 		(pts
-			(xy 240.03 110.49) (xy 241.3 110.49)
-		)
-		(stroke
-			(width 0)
-			(type default)
-		)
-	)
-	(wire
-		(pts
 			(xy 54.61 130.81) (xy 54.61 132.08)
 		)
@@
 	(wire
 		(pts
-			(xy 241.3 134.62) (xy 241.3 110.49)
-		)
-		(stroke
-			(width 0)
-			(type default)
-		)
-	)
-	(wire
-		(pts
 			(xy 254 120.65) (xy 261.62 120.65)
 		)
@@
 	(wire
 		(pts
-			(xy 256.54 134.62) (xy 241.3 134.62)
-		)
-		(stroke
-			(width 0)
-			(type default)
-		)
-	)
-	(wire
-		(pts
 			(xy 71.12 45.72) (xy 93.98 45.72)
 		)
@@
 	(wire
 		(pts
-			(xy 241.3 110.49) (xy 251.46 110.49)
+			(xy 240.03 110.49) (xy 251.46 110.49)
 		)
 		(stroke
@@
 					(unit 1)
 				)
+			)
+		)
+	)
+	(symbol
+		(lib_id "power:+3V3")
+		(at 256.54 134.62 90)
+		(unit 1)
+		(body_style 1)
+		(exclude_from_sim no)
+		(in_bom yes)
+		(on_board yes)
+		(in_pos_files yes)
+		(dnp no)
+		(property "Reference" "#PWR016"
+			(at 260.35 134.62 0)
+			(hide yes)
+			(show_name no)
+			(do_not_autoplace no)
+			(effects
+				(font
+					(size 1.27 1.27)
+				)
+			)
+		)
+		(property "Value" "+3V3"
+			(at 250.952 134.62 90)
+			(show_name no)
+			(do_not_autoplace no)
+			(effects
+				(font
+					(size 1.27 1.27)
+				)
+			)
+		)
+		(property "Footprint" ""
+			(at 256.54 134.62 0)
+			(hide yes)
+			(show_name no)
+			(do_not_autoplace no)
+			(effects
+				(font
+					(size 1.27 1.27)
+				)
+			)
+		)
+		(property "Datasheet" ""
+			(at 256.54 134.62 0)
+			(hide yes)
+			(show_name no)
+			(do_not_autoplace no)
+			(effects
+				(font
+					(size 1.27 1.27)
+				)
+			)
+		)
+		(property "Description" "Power symbol creates a global label with name \"+3V3\""
+			(at 256.54 134.62 0)
+			(hide yes)
+			(show_name no)
+			(do_not_autoplace no)
+			(effects
+				(font
+					(size 1.27 1.27)
+				)
+			)
+		)
+		(pin "1"
+		)
+		(instances
+			(project "Secondary Board"
+				(path "/148b448d-b722-497b-94de-5b72fb78c9d0"
+					(reference "#PWR016")
+					(unit 1)
+				)
